Commit message: Minor

File: data/robots/kuka_lwr/kuka_mobile_base_only.urdf (robot description, URDF)
Before this commit: robot kuka_lwr, 3 links, 2 joints
Links:
- added link empty_link_y
Joints:
- added joint joint_rotation_yaw: type continuous, parent empty_link_y, child base_link_robot, origin xyz=0 0 0 rpy=0 0 0, axis 0 0 1
- joint joint_translation_y: child base_link_robot -> empty_link_y
