Commit message: Add additional scenarios

File: data/robots/car.urdf (robot description, URDF)
Before this commit: robot car, 9 links, 8 joints
Joints:
- joint joint_translation_x: limit lower=-1.5 upper=1.5 effort=1 velocity=1 -> lower=-5.0 upper=5.0 effort=1 velocity=1
- joint joint_translation_y: limit lower=-1.5 upper=1.5 effort=1 velocity=1 -> lower=-5.0 upper=5.0 effort=1 velocity=1
