Commit message: Set up benchmarks

File: data/objects/uploads_files_2883707_warehouse6.urdf (robot description, URDF)
Before this commit: robot maze, 1 links, 0 joints
Links:
- link root: geometry collision mesh filename=uploads_files_2883707_warehouse6_simple.stl scale=0.5 0.5 0.5; visual mesh filename=uploads_files_2883707_warehouse6_simple.stl scale=0.5 0.5 0.5
